File: printer.kicad/printer.sch (KiCad schematic (older format))
At the start: 35 parts, among them J1 ZX_Spectrum_128K_expansion, J2 Conn_01x08_Male, J3 Conn_01x05_Male, J4 Conn_01x04_Male, U1 SN74AHC373, U2 SN74HCT00, U3 SN74AHCT02, U4 SN74AHC373, U5 XC6206PxxxMR, U6 STM32F103C8Tx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

Commit message: Start laying out the PCB
Parts:
- added unit 5 of U2
- added unit 5 of U3
Changed lines of the file:
@@
 L power:PWR_FLAG #FLG01
 U 1 1 5E1F67F9
-P -450 900
-F 0 "#FLG01" H -450 975 50  0001 C CNN
-F 1 "PWR_FLAG" H -450 1073 50  0000 C CNN
-F 2 "" H -450 900 50  0001 C CNN
-F 3 "~" H -450 900 50  0001 C CNN
-	1    -450 900
+P -2250 1500
+F 0 "#FLG01" H -2250 1575 50  0001 C CNN
+F 1 "PWR_FLAG" H -2250 1673 50  0000 C CNN
+F 2 "" H -2250 1500 50  0001 C CNN
+F 3 "~" H -2250 1500 50  0001 C CNN
+	1    -2250 1500
 	1    0    0    -1
 $EndComp
@@
 L power:GND #PWR01
 U 1 1 5E1F73ED
-P -450 900
-F 0 "#PWR01" H -450 650 50  0001 C CNN
-F 1 "GND" H -445 727 50  0000 C CNN
-F 2 "" H -450 900 50  0001 C CNN
-F 3 "" H -450 900 50  0001 C CNN
-	1    -450 900
+P -2250 1500
+F 0 "#PWR01" H -2250 1250 50  0001 C CNN
+F 1 "GND" H -2245 1327 50  0000 C CNN
+F 2 "" H -2250 1500 50  0001 C CNN
+F 3 "" H -2250 1500 50  0001 C CNN
+	1    -2250 1500
 	1    0    0    -1
 $EndComp
@@
 Wire Wire Line
 	4250 3800 4700 3800
+$Comp
+L 74xx:74HCT00 U2
+U 5 1 5DF4AABC
+P -1650 1000
+F 0 "U2" H -1650 1325 50  0000 C CNN
+F 1 "SN74HCT00" H -1650 1234 50  0000 C CNN
+F 2 "Package_SO:TSSOP-14_4.4x5mm_P0.65mm" H -1650 1000 50  0001 C CNN
+F 3 "https://www.ti.com/lit/ds/symlink/sn74hct00.pdf" H -1650 1000 50  0001 C CNN
+F 4 "C131694" H -1650 1000 50  0001 C CNN "LCSC"
+	5    -1650 1000
+	1    0    0    -1
+$EndComp
+$Comp
+L power:GND #PWR0101
+U 1 1 5DF5604C
+P -1650 1500
+F 0 "#PWR0101" H -1650 1250 50  0001 C CNN
+F 1 "GND" H -1645 1327 50  0000 C CNN
+F 2 "" H -1650 1500 50  0001 C CNN
+F 3 "" H -1650 1500 50  0001 C CNN
+	1    -1650 1500
+	1    0    0    -1
+$EndComp
+$Comp
+L power:+5V #PWR0102
+U 1 1 5DF7402F
+P -1650 500
+F 0 "#PWR0102" H -1650 350 50  0001 C CNN
+F 1 "+5V" H -1635 673 50  0000 C CNN
+F 2 "" H -1650 500 50  0001 C CNN
+F 3 "" H -1650 500 50  0001 C CNN
+	1    -1650 500
+	1    0    0    -1
+$EndComp
+$Comp
+L 74xx:74HCT02 U3
+U 5 1 5DF7B6F3
+P -1100 1000
+F 0 "U3" H -1100 1325 50  0000 C CNN
+F 1 "SN74AHCT02" H -1100 1234 50  0000 C CNN
+F 2 "Package_SO:TSSOP-14_4.4x5mm_P0.65mm" H -1100 1000 50  0001 C CNN
+F 3 "https://www.ti.com/lit/ds/symlink/sn74ahct02.pdf" H -1100 1000 50  0001 C CNN
+F 4 "C87964" H -1100 1000 50  0001 C CNN "LCSC"
+	5    -1100 1000
+	1    0    0    -1
+$EndComp
+$Comp
+L power:GND #PWR0103
+U 1 1 5DF8474F
+P -1100 1500
+F 0 "#PWR0103" H -1100 1250 50  0001 C CNN
+F 1 "GND" H -1095 1327 50  0000 C CNN
+F 2 "" H -1100 1500 50  0001 C CNN
+F 3 "" H -1100 1500 50  0001 C CNN
+	1    -1100 1500
+	1    0    0    -1
+$EndComp
+$Comp
+L power:+5V #PWR0104
+U 1 1 5DF84B95
+P -1100 500
+F 0 "#PWR0104" H -1100 350 50  0001 C CNN
+F 1 "+5V" H -1085 673 50  0000 C CNN
+F 2 "" H -1100 500 50  0001 C CNN
+F 3 "" H -1100 500 50  0001 C CNN
+	1    -1100 500
+	1    0    0    -1
+$EndComp
 $EndSCHEMATC
